File: PepeMatrix.sch (KiCad schematic (older format))
At the start: 56 parts

Commit message: Simple keyboard matrix. Trackball sensor pcb + gerbers
Parts:
- D1, D10, D11, D12, D13, D14, D15, D16, D17, D18, D19, D2, D20, D21, D22, D23, D24, D25, D26, D27, D28, D3, D4, D5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: renamed from D?; footprint (none) -> Diode_SMD:D_SOD-123
- SW1, SW10, SW11, SW12, SW13, SW14, SW15, SW16, SW17, SW18, SW19, SW2, SW20, SW21, SW22, SW23, SW24, SW25, SW26, SW27, SW28, SW3, SW4, SW5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: renamed from SW?; footprint (none) -> bankkis_lib:SW_MX_reversible
